Commit message: enable hrp2jsknts simulation(dashboard, HRP3Hand, Crane, realistic launchfiles+configfiles+setup.py)

File: hrpsys_gazebo_tutorials/robot_models/HRP2JSKNTS/HRP2JSKNTS.urdf.xacro (robot description, xacro)
@@ -6,4 +6,10 @@
       <robotname>HRP2JSKNTS</robotname>
       <controller>hrpsys_gazebo_configuration</controller>
+    </plugin>
+  </gazebo>
+  <gazebo>
+    <plugin filename="libIOBPlugin.so" name="hrp3hand_hrpsys_gazebo_plugin">
+      <robotname>HRP3HAND</robotname>
+      <controller>hrp3hand_hrpsys_gazebo_configuration</controller>
     </plugin>
   </gazebo>
@@ -46,41 +52,41 @@
   </gazebo>
   <!-- add Kinect plugin, link and joint without visual and collision -->
-  <joint name="xtion_joint" type="fixed">
-    <origin rpy="0 0 0" xyz="0.1120 0.0 0.1255"/>
-    <parent link="HEAD_LINK1"/>
-    <child link="xtion_link"/>
-  </joint>
-  <link name="xtion_link">
-    <inertial>
-      <mass value="0.200"/>
-      <origin rpy="0 0 0" xyz="0 0 0"/>
-      <inertia ixx="5.8083e-4" ixy="0" ixz="0" iyy="3.0833e-5" iyz="0" izz="5.9083e-4"/>
-    </inertial>
-  </link>
-  <joint name="xtion_depth_joint" type="fixed">
-    <origin rpy="0 0 0" xyz="0.0 0.049 0.0"/>
-    <parent link="xtion_link"/>
-    <child link="xtion_depth_frame"/>
-  </joint>
-  <link name="xtion_depth_frame"/>
-  <joint name="xtion_depth_optical_joint" type="fixed">
-    <origin rpy="-1.57079632679 0.0 -1.57079632679" xyz="0 0 0"/>
-    <parent link="xtion_depth_frame"/>
-    <child link="xtion_depth_optical_frame"/>
-  </joint>
-  <link name="xtion_depth_optical_frame"/>
-  <joint name="xtion_rgb_joint" type="fixed">
-    <origin rpy="0 0 0" xyz="0.0 0.022 0.0"/>
-    <parent link="xtion_link"/>
-    <child link="xtion_rgb_frame"/>
-  </joint>
-  <link name="xtion_rgb_frame"/>
-  <joint name="xtion_rgb_optical_joint" type="fixed">
-    <origin rpy="-1.57079632679 0.0 -1.57079632679" xyz="0 0 0"/>
-    <parent link="xtion_rgb_frame"/>
-    <child link="xtion_rgb_optical_frame"/>
-  </joint>
-  <link name="xtion_rgb_optical_frame"/>
-  <gazebo reference="xtion_depth_frame">
+  <!-- <joint name="xtion_joint" type="fixed"> -->
+  <!--   <origin rpy="0 0 0" xyz="0.1120 0.0 0.1255"/> -->
+  <!--   <parent link="HEAD_LINK1"/> -->
+  <!--   <child link="xtion_link"/> -->
+  <!-- </joint> -->
+  <!-- <link name="xtion_link"> -->
+  <!--   <inertial> -->
+  <!--     <mass value="0.200"/> -->
+  <!--     <origin rpy="0 0 0" xyz="0 0 0"/> -->
+  <!--     <inertia ixx="5.8083e-4" ixy="0" ixz="0" iyy="3.0833e-5" iyz="0" izz="5.9083e-4"/> -->
+  <!--   </inertial> -->
+  <!-- </link> -->
+  <!-- <joint name="xtion_depth_joint" type="fixed"> -->
+  <!--   <origin rpy="0 0 0" xyz="0.0 0.049 0.0"/> -->
+  <!--   <parent link="xtion_link"/> -->
+  <!--   <child link="xtion_depth_frame"/> -->
+  <!-- </joint> -->
+  <!-- <link name="xtion_depth_frame"/> -->
+  <!-- <joint name="xtion_depth_optical_joint" type="fixed"> -->
+  <!--   <origin rpy="-1.57079632679 0.0 -1.57079632679" xyz="0 0 0"/> -->
+  <!--   <parent link="xtion_depth_frame"/> -->
+  <!--   <child link="xtion_depth_optical_frame"/> -->
+  <!-- </joint> -->
+  <!-- <link name="xtion_depth_optical_frame"/> -->
+  <!-- <joint name="xtion_rgb_joint" type="fixed"> -->
+  <!--   <origin rpy="0 0 0" xyz="0.0 0.022 0.0"/> -->
+  <!--   <parent link="xtion_link"/> -->
+  <!--   <child link="xtion_rgb_frame"/> -->
+  <!-- </joint> -->
+  <!-- <link name="xtion_rgb_frame"/> -->
+  <!-- <joint name="xtion_rgb_optical_joint" type="fixed"> -->
+  <!--   <origin rpy="-1.57079632679 0.0 -1.57079632679" xyz="0 0 0"/> -->
+  <!--   <parent link="xtion_rgb_frame"/> -->
+  <!--   <child link="xtion_rgb_optical_frame"/> -->
+  <!-- </joint> -->
+  <!-- <link name="xtion_rgb_optical_frame"/> -->
+  <gazebo reference="camera_depth_frame">
     <sensor name="xtion" type="depth">
       <update_rate>20</update_rate>
@@ -100,10 +106,10 @@
         <alwaysOn>true</alwaysOn>
         <updateRate>20</updateRate>
-        <imageTopicName>xtion/rgb/image_raw</imageTopicName>
-        <cameraInfoTopicName>xtion/rgb/camera_info</cameraInfoTopicName>
-        <depthImageTopicName>xtion/depth/image_raw</depthImageTopicName>
-        <depthImageCameraInfoTopicName>xtion/depth/camera_info</depthImageCameraInfoTopicName>
-        <pointCloudTopicName>xtion/depth/points</pointCloudTopicName>
-        <frameName>xtion_depth_optical_frame</frameName>
+        <imageTopicName>camera_remote/rgb/image_raw</imageTopicName>
+        <cameraInfoTopicName>camera_remote/rgb/camera_info</cameraInfoTopicName>
+        <depthImageTopicName>camera_remote/depth/image_raw</depthImageTopicName>
+        <depthImageCameraInfoTopicName>camera_remote/depth/camera_info</depthImageCameraInfoTopicName>
+        <pointCloudTopicName>camera_remote/depth/points</pointCloudTopicName>
+        <frameName>camera_depth_optical_frame</frameName>
         <distortion_k1>0.0</distortion_k1>
         <distortion_k2>0.0</distortion_k2>
@@ -146,3 +152,16 @@
     </plugin>
   </gazebo>
+  <gazebo>
+    <plugin filename="libCranePlugin.so" name="crane_plugin" >
+      <objname>HRP2JSKNTS</objname>
+      <linkname>CHEST_LINK1</linkname>
+      <liftheight>1.2</liftheight>
+      <lowerheight>0.5</lowerheight>
+      <liftvelocity>0.1</liftvelocity>
+      <lowervelocity>0.03</lowervelocity>
+      <pgain>5000</pgain>
+      <dgain>1000</dgain>
+      <damp>10000</damp>
+    </plugin>
+  </gazebo>
 </robot>
