Commit message: fix cannot set contolloer bag

File: hrpsys_gazebo_tutorials/robot_models/HRP2JSKNTS/HRP2JSKNTS_with_kannna.urdf.xacro (robot description, xacro)
@@ -70,11 +70,11 @@
     </inertial>
   </link>
-  <joint name="kannna_to_hand" type="revolute">
+  <joint name="kannna_to_hand" type="fixed">
+    <origin rpy="0 0 0" xyz="0 0 0"/>
     <parent link="LARM_LINK6"/>
     <child link="kannna"/>
-    <origin xyz="0 0 0" rpy="0 0 0"/>
-    <axis xyz="0 1 0"/>
-    <limit effort="1000" lower="-0.261799" upper="1.6057" velocity="10.0"/>
-    <dynamics friction="10000"/>
+    <!-- <axis xyz="0 1 0"/> -->
+    <!-- <limit effort="1000" lower="-0.261799" upper="1.6057" velocity="10.0"/> -->
+    <!-- <dynamics friction="10000"/> -->
   </joint>
   <gazebo reference="kannna">
@@ -85,5 +85,5 @@
     <mu2>1.0</mu2>
   </gazebo>
-  <!-- add Kinect plugin, link and joint without visual and collision -->
+    <!-- add Kinect plugin, link and joint without visual and collision -->
   <!-- <joint name="xtion_joint" type="fixed"> -->
   <!--   <origin rpy="0 0 0" xyz="0.1120 0.0 0.1255"/> -->
