Commit message: add table, wooded board, and robot model with kannna

File: hrpsys_gazebo_tutorials/robot_models/HRP2JSKNTS_with_kannna/HRP2JSKNTS_with_kannna.urdf.xacro (robot description, xacro)
@@ -50,4 +50,38 @@
   <gazebo reference="RARM_JOINT6">
     <provideFeedback>1</provideFeedback>
+  </gazebo>
+  <!-- add kannna -->
+  <link name="kannna">
+    <visual>
+      <geometry>
+	<box size="0.15 0.055 0.025"/>
+      </geometry>
+      <origin xyz="0.02 0.025 -0.23" ryp="0 0 0"/>
+    </visual>
+    <collision>
+      <geometry>
+	<box size="0.15 0.055 0.025"/>
+      </geometry>
+      <origin xyz="0.02 0.025 -0.23" ryp="0 0 0"/>
+    </collision>
+    <inertial>
+      <mass value="0.2"/>
+      <inertia ixx="1e-3" ixy="0.0" ixz="0.0" iyy="1e-3" iyz="0.0" izz="1e-3"/>
+    </inertial>
+  </link>
+  <joint name="kannna_to_hand" type="revolute">
+    <parent link="LARM_LINK6"/>
+    <child link="kannna"/>
+    <origin xyz="0 0 0" rpy="0 0 0"/>
+    <axis xyz="0 1 0"/>
+    <limit effort="1000" lower="-0.261799" upper="1.6057" velocity="10.0"/>
+    <dynamics friction="10000"/>
+  </joint>
+  <gazebo reference="kannna">
+    <material>Gazebo/WoodFloor</material>
+  </gazebo>
+  <gazebo refetence="kannna">
+    <mu1>1.0</mu1>
+    <mu2>1.0</mu2>
   </gazebo>
   <!-- add Kinect plugin, link and joint without visual and collision -->
