Commit message: change kannna-table and wodden-board static to the world

File: hrpsys_gazebo_tutorials/environment_models/kannna-table/model.urdf (robot description, URDF)
Before this commit: robot room73b2-karimoku-table, 1 links, 0 joints
Links:
- link nil_link: mass 20.0 -> 100.0

File: hrpsys_gazebo_tutorials/environment_models/wooden_board/model.urdf (robot description, URDF)
Before this commit: robot simple_box, 1 links, 0 joints
Links:
- link nil_link: mass 10 -> 100.0; geometry collision box size=0.6 1.5 0.01; visual box size=0.6 1.5 0.01

File: hrpsys_gazebo_tutorials/robot_models/kannna_HRP2JSKNTS/HRP2JSKNTS_with_kannna.urdf.xacro (robot description, xacro)
@@ -81,5 +81,10 @@
     <material>Gazebo/WoodFloor</material>
   </gazebo>
-  <gazebo refetence="kannna">
+  <gazebo reference="kannna">
+    <kp>1400000.0</kp>
+    <kd>280.0</kd>
+    <fdir1>1 0 0</fdir1>
+    <maxVel>10.0</maxVel>
+    <minDepth>0.00</minDepth>
     <mu1>1.0</mu1>
     <mu2>1.0</mu2>
